File: 4_switch_pcb/4_switch_pcb.kicad_pcb (KiCad board)
At the start: 2 copper layers, 27 parts, among them J1 USB_B_Micro, J2 AVR-ISP-6, J3 Conn_01x03_Pin, SW1 SW_Push, SW2 SW_Push, SW3 SW_Push, SW4 SW_Push, SW5 SW_Push, U1 ATmega32U4-A, Y1 Crystal 16Mhz

Commit message: component alignement
Parts:
- C1, C2, C3, C4, C5, C6, C7, C8, C9, D1, D2, D3, D4, J1, J2, J3, R1, R2, R3, R4, SW1, U1, Y1: moved to B.Cu
- SW2, SW3, SW4, SW5: footprint Button_Switch_SMD:SW_SPST_TL3342 -> Button_Switch_Keyboard:SW_Cherry_MX_1.00u_PCB
- moved SW1 62.0 mm to (183.4, 88.1), turned to 180 degrees
- moved C8 47.3 mm to (173.8, 71.4), turned to -90 degrees
- moved C4 43.3 mm to (173.8, 83.3), turned to -90 degrees
- moved C1 42.5 mm to (169.1, 88.1), turned to -90 degrees
- moved C6 42.4 mm to (167.7, 64.3), turned to 180 degrees
- moved J1 39.0 mm to (182.6, 77.0), turned to -90 degrees
- moved C3 34.3 mm to (163.0, 64.3), turned to 180 degrees
- moved R3 32.4 mm to (174.8, 75.5), turned to 180 degrees
- moved R4 32.2 mm to (174.8, 79.0), turned to 180 degrees
- moved J2 32.1 mm to (180.8, 66.7), turned to -90 degrees
- moved SW4 31.7 mm to (119.5, 61.6)
- moved C5 30.7 mm to (155.8, 64.3), turned to 180 degrees
- moved C2 30.5 mm to (157.2, 88.1), turned to -90 degrees
- moved C9 30.5 mm to (152.4, 72.5), turned to -90 degrees
- moved R2 29.0 mm to (174.8, 89.0), turned to -90 degrees
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Routing:
- net Net-(U1-XTAL2): track 0.00 -> 10.5 mm
- net Net-(U1-XTAL1): track 0.00 -> 10.1 mm
- added copper zone on F.Cu, net GND
Other:
- board outline added: 84.5 x 43.5 mm

Commit message: add base of routing
Parts:
- removed Y1: Crystal 16Mhz, user:crystal_FA238-TSX3225
- added X1: 16 MHZ, user:crystal_FA238-TSX3225, B.Cu at (162.0, 88.0)
- C8: value 100nF -> 4.7uF
- moved R1 34.1 mm to (185.2, 61.8), turned to 90 degrees
- moved R2 32.3 mm to (151.0, 67.2), turned to 90 degrees
- moved SW1 27.6 mm to (176.0, 61.5)
- moved C4 23.4 mm to (152.0, 74.8), turned to 90 degrees
- moved C3 22.6 mm to (175.0, 83.5)
- moved J2 22.6 mm to (179.2, 89.2)
- moved C9 22.5 mm to (174.8, 70.2), turned to 180 degrees
- moved J3 14.1 mm to (161.6, 60.0)
- moved C8 9.37 mm to (183.0, 69.5), turned to 0 degrees
- moved R4 3.75 mm to (174.8, 75.2)
- moved R3 3.50 mm to (174.8, 79.0)
- moved C1 1.00 mm to (168.1, 88.1)
- moved C2 1.00 mm to (156.2, 88.1)
- moved C6 0.97 mm to (166.8, 64.3)
Routing:
- net VCC: track 0.00 -> 68.7 mm
- net Net-(U1-XTAL1): track 10.1 -> 11.8 mm
- net Net-(U1-XTAL2): track 10.5 -> 11.6 mm

Commit message: base of pcb edition
Parts:
- moved R3 2.85 mm to (177.2, 77.6)
- moved R4 2.85 mm to (177.2, 73.8)
- moved C9 1.20 mm to (174.9, 69.1)
- moved C3 0.43 mm to (175.0, 83.1)
Routing:
- net Net-(U1-~{RESET}): track 0.00 -> 28.9 mm
- net Net-(U1-UCAP): track 0.00 -> 14.0 mm
- net Net-(U1-VBUS): track 0.00 -> 12.4 mm, vias 0 -> 2
- net Net-(U1-D+): track 0.00 -> 9.82 mm
- net Net-(U1-D-): track 0.00 -> 8.60 mm
- net Net-(J1-D-): track 0.00 -> 5.37 mm
- net Net-(J1-D+): track 0.00 -> 4.62 mm
- net VCC: track 68.7 -> 69.9 mm, vias 0 -> 2
Changed lines of the file:
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@@
   )
   (footprint "Capacitor_SMD:C_0805_2012Metric_Pad1.18x1.45mm_HandSolder" (layer "B.Cu")
-    (at 174.75 70.25 180)
+    (at 174.86875 69.05625 180)
     (descr "Capacitor SMD 0805 (2012 Metric), square (rectangular) end terminal, IPC_7351 nominal with elongated pad for handsoldering. (Body size source: IPC-SM-782 page 76, https://www.pcb-3d.com/wordpress/wp-content/uploads/ipc-sm-782a_amendment_1_and_2.pdf, https://docs.google.com/spreadsheets/d/1BsfQQcO9C6DZCsRaXUlFlo91Tg2WpOkGARC1WS5S8t0/edit?usp=sharing), generated with kicad-footprint-generator")
     (tags "capacitor handsolder")
@@
   )
   (footprint "Resistor_SMD:R_0805_2012Metric_Pad1.20x1.40mm_HandSolder" (layer "B.Cu")
-    (at 174.75 75.25 180)
+    (at 177.2125 73.81875 180)
     (descr "Resistor SMD 0805 (2012 Metric), square (rectangular) end terminal, IPC_7351 nominal with elongated pad for handsoldering. (Body size source: IPC-SM-782 page 72, https://www.pcb-3d.com/wordpress/wp-content/uploads/ipc-sm-782a_amendment_1_and_2.pdf), generated with kicad-footprint-generator")
     (tags "resistor handsolder")
@@
   )
   (footprint "Capacitor_SMD:C_0805_2012Metric_Pad1.18x1.45mm_HandSolder" (layer "B.Cu")
-    (at 174.9625 83.5 180)
+    (at 175.04375 83.08125 180)
     (descr "Capacitor SMD 0805 (2012 Metric), square (rectangular) end terminal, IPC_7351 nominal with elongated pad for handsoldering. (Body size source: IPC-SM-782 page 76, https://www.pcb-3d.com/wordpress/wp-content/uploads/ipc-sm-782a_amendment_1_and_2.pdf, https://docs.google.com/spreadsheets/d/1BsfQQcO9C6DZCsRaXUlFlo91Tg2WpOkGARC1WS5S8t0/edit?usp=sharing), generated with kicad-footprint-generator")
     (tags "capacitor handsolder")
@@
   )
   (footprint "Resistor_SMD:R_0805_2012Metric_Pad1.20x1.40mm_HandSolder" (layer "B.Cu")
-    (at 174.75 79 180)
+    (at 177.2125 77.56875 180)
     (descr "Resistor SMD 0805 (2012 Metric), square (rectangular) end terminal, IPC_7351 nominal with elongated pad for handsoldering. (Body size source: IPC-SM-782 page 72, https://www.pcb-3d.com/wordpress/wp-content/uploads/ipc-sm-782a_amendment_1_and_2.pdf), generated with kicad-footprint-generator")
     (tags "resistor handsolder")
@@
   (segment (start 157.305882 88.212132) (end 160.656497 88.212132) (width 0.25) (layer "B.Cu") (net 3))
   (segment (start 160.656497 84.043503) (end 161.925 82.775) (width 0.25) (layer "B.Cu") (net 3))
+  (segment (start 168.83125 83.08125) (end 166.55 80.8) (width 0.25) (layer "B.Cu") (net 4))
+  (segment (start 174.00625 83.08125) (end 168.83125 83.08125) (width 0.25) (layer "B.Cu") (net 4))
+  (segment (start 166.625 76.2) (end 167.625 76.2) (width 0.25) (layer "B.Cu") (net 4))
+  (segment (start 166.55 76.275) (end 166.625 76.2) (width 0.25) (layer "B.Cu") (net 4))
+  (segment (start 166.55 80.8) (end 166.55 76.275) (width 0.25) (layer "B.Cu") (net 4))
+  (segment (start 154.27 75.85) (end 165.31 75.85) (width 0.25) (layer "F.Cu") (net 5))
+  (segment (start 165.31 75.85) (end 166.05 75.11) (width 0.25) (layer "F.Cu") (net 5))
+  (via (at 154.27 75.85) (size 0.8) (drill 0.4) (layers "F.Cu" "B.Cu") (net 5))
+  (via (at 166.05 75.11) (size 0.8) (drill 0.4) (layers "F.Cu" "B.Cu") (net 5))
+  (segment (start 154.245 75.825) (end 154.27 75.85) (width 0.25) (layer "B.Cu") (net 5))
+  (segment (start 152 75.825) (end 154.245 75.825) (width 0.25) (layer "B.Cu") (net 5))
+  (segment (start 164.325 80.945) (end 164.325 81.9) (width 0.25) (layer "B.Cu") (net 5))
+  (segment (start 165.925 71.5) (end 164.975 72.45) (width 0.25) (layer "B.Cu") (net 5))
+  (segment (start 152.085 75.825) (end 152.28 76.02) (width 0.25) (layer "B.Cu") (net 5))
   (segment (start 152.4 79.925) (end 152.925 79.4) (width 0.25) (layer "B.Cu") (net 5))
   (segment (start 152.925 79.4) (end 156.225 79.4) (width 0.25) (layer "B.Cu") (net 5))
-  (segment (start 164.325 78.575) (end 164.325 81.9) (width 0.25) (layer "B.Cu") (net 5))
-  (segment (start 155.15 72.675) (end 155.15 71.6) (width 0.25) (layer "B.Cu") (net 5))
+  (segment (start 164.975 72.45) (end 163.68 72.45) (width 0.25) (layer "B.Cu") (net 5))
+  (segment (start 166.625 73) (end 167.625 73) (width 0.25) (layer "B.Cu") (net 5))
+  (segment (start 181.9625 69.5) (end 176.35 69.5) (width 0.25) (layer "B.Cu") (net 5))
+  (segment (start 166.05 75.11) (end 166.05 73.575) (width 0.25) (layer "B.Cu") (net 5))
+  (segment (start 163.29 72.84) (end 163.29 79.91) (width 0.25) (layer "B.Cu") (net 5))
   (segment (start 182.6 75.4) (end 182.6 70.1375) (width 0.25) (layer "B.Cu") (net 5))
+  (segment (start 152.085 75.825) (end 152 75.825) (width 0.25) (layer "B.Cu") (net 5))
   (segment (start 181.9625 66.0375) (end 181.9625 69.5) (width 0.25) (layer "B.Cu") (net 5))
-  (segment (start 157.35 71.6) (end 164.325 78.575) (width 0.25) (layer "B.Cu") (net 5))
   (segment (start 165.925 66.15625) (end 165.925 70.5) (width 0.25) (layer "B.Cu") (net 5))
-  (segment (start 152 75.825) (end 155.15 72.675) (width 0.25) (layer "B.Cu") (net 5))
-  (segment (start 155.15 71.6) (end 157.35 71.6) (width 0.25) (layer "B.Cu") (net 5))
+  (segment (start 163.29 79.91) (end 164.325 80.945) (width 0.25) (layer "B.Cu") (net 5))
+  (segment (start 165.925 70.5) (end 165.925 71.5) (width 0.25) (layer "B.Cu") (net 5))
   (segment (start 156.85625 64.29375) (end 157.925 65.3625) (width 0.25) (layer "B.Cu") (net 5))
-  (segment (start 178.4625 73) (end 167.625 73) (width 0.25) (layer "B.Cu") (net 5))
+  (segment (start 163.68 72.45) (end 163.29 72.84) (width 0.25) (layer "B.Cu") (net 5))
   (segment (start 157.925 65.3625) (end 157.925 70.5) (width 0.25) (layer "B.Cu") (net 5))
   (segment (start 182.6 70.1375) (end 181.9625 69.5) (width 0.25) (layer "B.Cu") (net 5))
-  (segment (start 181.9625 69.5) (end 178.4625 73) (width 0.25) (layer "B.Cu") (net 5))
+  (segment (start 176.35 69.5) (end 175.90625 69.05625) (width 0.25) (layer "B.Cu") (net 5))
+  (segment (start 166.05 73.575) (end 166.625 73) (width 0.25) (layer "B.Cu") (net 5))
   (segment (start 167.7875 64.29375) (end 165.925 66.15625) (width 0.25) (layer "B.Cu") (net 5))
   (segment (start 185.25 62.75) (end 181.9625 66.0375) (width 0.25) (layer "B.Cu") (net 5))
+  (segment (start 170.8 72.84) (end 170.8 76.95) (width 0.25) (layer "F.Cu") (net 6))
+  (segment (start 170.8 76.95) (end 170.83 76.98) (width 0.25) (layer "F.Cu") (net 6))
+  (via (at 170.8 72.84) (size 0.8) (drill 0.4) (layers "F.Cu" "B.Cu") (net 6))
+  (via (at 170.83 76.98) (size 0.8) (drill 0.4) (layers "F.Cu" "B.Cu") (net 6))
+  (segment (start 170.81 77) (end 167.625 77) (width 0.25) (layer "B.Cu") (net 6))
+  (segment (start 170.8 72.0875) (end 170.8 72.84) (width 0.25) (layer "B.Cu") (net 6))
+  (segment (start 170.83 76.98) (end 170.81 77) (width 0.25) (layer "B.Cu") (net 6))
+  (segment (start 173.83125 69.05625) (end 170.8 72.0875) (width 0.25) (layer "B.Cu") (net 6))
+  (segment (start 180.59375 76.2) (end 178.2125 73.81875) (width 0.25) (layer "B.Cu") (net 13))
+  (segment (start 182.6 76.2) (end 180.59375 76.2) (width 0.25) (layer "B.Cu") (net 13))
+  (segment (start 182.6 77) (end 178.78125 77) (width 0.25) (layer "B.Cu") (net 14))
+  (segment (start 178.78125 77) (end 178.2125 77.56875) (width 0.25) (layer "B.Cu") (net 14))
+  (segment (start 165.125 73.085) (end 165.125 81.9) (width 0.25) (layer "B.Cu") (net 23))
+  (segment (start 166.55 71.66) (end 165.125 73.085) (width 0.25) (layer "B.Cu") (net 23))
+  (segment (start 182.6 63.4) (end 185.25 60.75) (width 0.25) (layer "B.Cu") (net 23))
+  (segment (start 166.55 69.7) (end 166.55 71.66) (width 0.25) (layer "B.Cu") (net 23))
+  (segment (start 172.85 63.4) (end 166.55 69.7) (width 0.25) (layer "B.Cu") (net 23))
+  (segment (start 179.15 63.4) (end 182.6 63.4) (width 0.25) (layer "B.Cu") (net 23))
+  (segment (start 173.24375 74.6) (end 167.625 74.6) (width 0.25) (layer "B.Cu") (net 25))
+  (segment (start 176.2125 77.56875) (end 173.24375 74.6) (width 0.25) (layer "B.Cu") (net 25))
+  (segment (start 176.2125 73.81875) (end 176.19375 73.8) (width 0.25) (layer "B.Cu") (net 26))
+  (segment (start 176.19375 73.8) (end 167.625 73.8) (width 0.25) (layer "B.Cu") (net 26))
   (zone (net 2) (net_name "GND") (layer "F.Cu") (hatch edge 0.5)
     (connect_pads (clearance 0.5))

Commit message: pcb finish
Parts:
- J3: footprint Connector_PinHeader_1.00mm:PinHeader_1x03_P1.00mm_Vertical_SMD_Pin1Right -> Connector_PinHeader_1.00mm:PinHeader_1x03_P1.00mm_Vertical
- moved D2 22.1 mm to (116.8, 71.1)
- moved D1 19.7 mm to (137.2, 71.1)
- moved J3 3.84 mm to (160.1, 63.5), turned to -90 degrees
- moved J1 0.28 mm to (182.9, 77.0)
Routing:
- net /col0: track 0.00 -> 77.4 mm, vias 0 -> 1
- net /row1: track 0.00 -> 71.5 mm
- net GND: track 0.00 -> 66.7 mm, vias 0 -> 5
- net /row0: track 0.00 -> 51.7 mm
- net /col1: track 0.00 -> 51.3 mm
- net VCC: track 69.9 -> 119.8 mm, vias 2 -> 3
- net Net-(J2-MOSI): track 0.00 -> 23.8 mm
- net Net-(J2-~{RST}): track 0.00 -> 22.8 mm, vias 0 -> 2
- net Net-(J2-SCK): track 0.00 -> 22.3 mm
- net Net-(J2-MISO): track 0.00 -> 19.1 mm
- net Net-(D4-A): track 0.00 -> 10.8 mm
- net Net-(D3-A): track 0.00 -> 10.6 mm
- net Net-(D2-A): track 0.00 -> 10.0 mm
- net Net-(D1-A): track 0.00 -> 9.76 mm
- net Net-(J3-Pin_3): track 0.00 -> 7.47 mm
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- added copper zone on B.Cu, net GND
Other:
- board size 84.5 x 43.5 mm -> 84.6 x 39.4 mm
